Commit message: fixed the gazebo model

File: code/hal_description/urdf/hal.urdf (robot description, URDF)
Before this commit: robot hal, 9 links, 8 joints
Links:
- link back_ball: geometry collision sphere radius=0.05; visual sphere radius=0.05
- link body: geometry collision box size=0.8 0.3 0.1; visual box size=0.8 0.3 0.1
- link left_wheel: geometry collision cylinder length=0.1 radius=0.1; visual cylinder length=0.1 radius=0.1
- link right_wheel: geometry collision cylinder length=0.1 radius=0.1; visual cylinder length=0.1 radius=0.1
Joints:
- removed joint base_footprint_to_back_ball
- added joint body_to_back_ball: type floating, parent body, child back_ball, origin xyz=-0.4 0 -0.05 rpy=0 0 0
- joint base_footprint_to_base_link: origin xyz=0 0 0.12 rpy=0 0 0 -> xyz=0 0 0.2 rpy=0 0 0
- joint base_footprint_to_body: origin xyz=0 0 0.12 rpy=0 0 0 -> xyz=0 0 0.2 rpy=0 0 0
- joint base_footprint_to_center_camera: origin xyz=0.03302 0 1.7145 rpy=0 0 0 -> xyz=0.4 0 0.5 rpy=0 0 0
- joint base_footprint_to_lidar: origin xyz=0.4572 0 0.9525 rpy=0 0 0 -> xyz=0.3 0 0.35 rpy=0 0 0
- joint body_to_left_wheel: origin xyz=0 0 -0.32004 rpy=0 0 0 -> xyz=0.2 -0.2 0 rpy=1.5708 0 0
- joint body_to_right_wheel: origin xyz=0 0 0.32004 rpy=0 0 0 -> xyz=0.2 0.2 0 rpy=1.5708 0 0
